File: tps65987d/Type-C Test Fixture (TPS65987D)_v3.brd (EAGLE design)
At the start: 74.4 x 38.6 mm, 195 parts, among them J1 105450-0101, J2 105450-0101, J3 105450-0101, J4 640456-4, J5 5040500491, Q1 AO3400A, Q10 AO3400A, Q11 AO3400A, Q12 AO3400A, Q13 AO3400A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

Commit message: Fix 5V FB resistors
Parts:
- removed R43: 332k, rcl:R0402
- removed R44: 1M, rcl:R0402
Connections:
- removed net FB: R43.1, R44.1, U10.6
- net +5V: now also U10.6; no longer R44.2
- net GND: no longer R43.2
Routing:
- net FB: track 2.81 -> 0.00 mm
- net REG_EN: track 25.3 -> 26.2 mm
- net GND: track 113.7 -> 113.1 mm, vias 167 -> 166
Changed lines of the file:
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@@
 <attribute name="VALUE" x="5.662" y="21.2" size="0.6096" layer="27" font="vector" ratio="20" rot="R90" align="top-center"/>
 </element>
-<element name="R43" library="rcl" package="R0402" package3d_urn="urn:adsk.eagle:package:23547/3" value="332k" x="3.7" y="20.3" smashed="yes" rot="R90">
-<attribute name="NAME" x="3.435" y="22.235" size="0.4064" layer="25" font="vector" rot="R270"/>
-<attribute name="POPULARITY" value="0" x="3.7" y="20.3" size="1.778" layer="27" rot="R90" display="off"/>
-<attribute name="SPICEPREFIX" value="R" x="3.7" y="20.3" size="1.778" layer="27" rot="R90" display="off"/>
-<attribute name="VALUE" x="5.605" y="19.665" size="1.27" layer="27" rot="R90"/>
-</element>
-<element name="R44" library="rcl" package="R0402" package3d_urn="urn:adsk.eagle:package:23547/3" value="1M" x="2.7" y="20.3" smashed="yes" rot="R90">
-<attribute name="NAME" x="2.435" y="22.235" size="0.4064" layer="25" font="vector" rot="R270"/>
-<attribute name="POPULARITY" value="0" x="2.7" y="20.3" size="1.778" layer="27" rot="R90" display="off"/>
-<attribute name="SPICEPREFIX" value="R" x="2.7" y="20.3" size="1.778" layer="27" rot="R90" display="off"/>
-<attribute name="VALUE" x="4.605" y="19.665" size="1.27" layer="27" rot="R90"/>
-</element>
 <element name="R48" library="rcl" package="R0402" package3d_urn="urn:adsk.eagle:package:23547/3" value="1M" x="1.8" y="20.3" smashed="yes" rot="R270">
 <attribute name="NAME" x="1.535" y="22.235" size="0.4064" layer="25" font="vector" rot="R270"/>
@@
 <contactref element="C67" pad="2"/>
 <contactref element="C68" pad="2"/>
-<contactref element="R43" pad="2"/>
 <contactref element="U10" pad="4"/>
 <contactref element="R48" pad="1"/>
@@
 <wire x1="58.2" y1="11.9" x2="58.8" y2="11.9" width="0.3048" layer="1"/>
 <via x="58.8" y="11.9" extent="1-16" drill="0.2"/>
-<wire x1="3.7" y1="20.8" x2="3.7" y2="21.4" width="0.3048" layer="1"/>
-<via x="3.7" y="21.4" extent="1-16" drill="0.2"/>
 <via x="48.39" y="17.84" extent="1-16" drill="0.3"/>
 <wire x1="48.39" y1="17.84" x2="48.39" y2="17.221840625" width="0.3048" layer="1"/>
@@
 <contactref element="C61" pad="1"/>
 <contactref element="C62" pad="1"/>
-<contactref element="R44" pad="2"/>
 <contactref element="U13" pad="4"/>
 <contactref element="C74" pad="1"/>
@@
 <wire x1="56.1" y1="10.8" x2="55.8" y2="10.8" width="0.3048" layer="1"/>
 <via x="55.8" y="10.8" extent="1-16" drill="0.2"/>
-<wire x1="2.7" y1="20.8" x2="2.7" y2="21.4" width="0.2032" layer="1"/>
-<via x="2.7" y="21.4" extent="1-16" drill="0.2"/>
-<via x="1.2" y="14.4" extent="1-16" drill="0.2"/>
 <via x="0.6" y="14.4" extent="1-16" drill="0.2"/>
 <via x="0.6" y="13.8" extent="1-16" drill="0.2"/>
@@
 <via x="0.6" y="10.4" extent="1-16" drill="0.2"/>
 <via x="1.2" y="10.4" extent="1-16" drill="0.2"/>
-<wire x1="2.7" y1="21.4" x2="1.2" y2="19.9" width="0.2032" layer="16"/>
-<wire x1="1.2" y1="19.9" x2="1.2" y2="14.4" width="0.2032" layer="16"/>
 <via x="50.6" y="21.2" extent="1-16" drill="0.2"/>
 <wire x1="3.1" y1="11" x2="3.1" y2="10.2" width="0.3048" layer="1"/>
@@
 <wire x1="-1.2" y1="10" x2="-1.2" y2="11.8" width="1.27" layer="1"/>
 <wire x1="-5.8" y1="5.4" x2="-1.2" y2="10" width="1.27" layer="1"/>
+<contactref element="U10" pad="6"/>
+<wire x1="3.2207125" y1="17.90355625" x2="3.2207125" y2="18.8" width="0.2032" layer="1"/>
+<via x="3.2207125" y="18.8" extent="1-16" drill="0.2"/>
+<wire x1="3.2207125" y1="18.8" x2="2" y2="18.8" width="0.2032" layer="16"/>
+<wire x1="1.6" y1="15" x2="2" y2="14.6" width="0.2032" layer="16"/>
+<wire x1="2" y1="18.8" x2="1.6" y2="18.4" width="0.2032" layer="16"/>
+<wire x1="1.6" y1="18.4" x2="1.6" y2="15" width="0.2032" layer="16"/>
+<wire x1="3.1" y1="13.8" x2="3.1" y2="14.6" width="0.2032" layer="1"/>
+<via x="3.1" y="14.6" extent="1-16" drill="0.2"/>
+<wire x1="2" y1="14.6" x2="3.1" y2="14.6" width="0.2032" layer="16"/>
 </signal>
 <signal name="GPIO12">
@@
 <wire x1="40.4" y1="21.2" x2="42" y2="19.6" width="0.4064" layer="1"/>
 <wire x1="26.6" y1="26" x2="26.65" y2="26.05" width="0.4064" layer="1"/>
-<wire x1="39.8" y1="21.8" x2="39.8" y2="24" width="0.4064" layer="1"/>
-<wire x1="44.2" y1="32" x2="44.2" y2="32.8" width="0.4064" layer="1"/>
+<wire x1="39.8" y1="21.8" x2="39.8" y2="24.6" width="0.4064" layer="1"/>
 <wire x1="44.2" y1="32.8" x2="45.2" y2="33.8" width="0.4064" layer="1"/>
 <wire x1="45.863" y1="33.8" x2="46.613" y2="34.55" width="0.4064" layer="1"/>
-<wire x1="39.8" y1="24" x2="41.8" y2="26" width="0.4064" layer="1"/>
-<wire x1="41.8" y1="26" x2="41.8" y2="29.6" width="0.4064" layer="1"/>
-<wire x1="41.8" y1="29.6" x2="44.2" y2="32" width="0.4064" layer="1"/>
+<wire x1="39.8" y1="24.6" x2="41.6" y2="26.4" width="0.4064" layer="1"/>
+<wire x1="41.6" y1="26.4" x2="41.6" y2="29.4" width="0.4064" layer="1"/>
 <wire x1="45.2" y1="33.8" x2="45.863" y2="33.8" width="0.4064" layer="1"/>
 <wire x1="39.8" y1="21.8" x2="40.4" y2="21.2" width="0.4064" layer="1"/>
@@
 <wire x1="20.6" y1="22.2" x2="24.4" y2="26" width="0.6096" layer="1"/>
 <wire x1="21.92" y1="18.72" x2="20.6" y2="17.4" width="0.508" layer="1"/>
+<wire x1="41.6" y1="29.4" x2="44.2" y2="32" width="0.4064" layer="1"/>
+<wire x1="44.2" y1="32" x2="44.2" y2="32.8" width="0.4064" layer="1"/>
 </signal>
 <signal name="N$21">
@@
 <via x="4.2" y="7.55" extent="1-16" drill="0.2"/>
 </signal>
-<signal name="FB">
-<contactref element="U10" pad="6"/>
-<contactref element="R44" pad="1"/>
-<contactref element="R43" pad="1"/>
-<wire x1="3.2207125" y1="17.90355625" x2="3.2207125" y2="19.3207125" width="0.2032" layer="1"/>
-<wire x1="3.2207125" y1="19.3207125" x2="3.7" y2="19.8" width="0.2032" layer="1"/>
-<wire x1="3.2207125" y1="19.3207125" x2="2.741425" y2="19.8" width="0.2032" layer="1"/>
-<wire x1="2.741425" y1="19.8" x2="2.7" y2="19.8" width="0.2032" layer="1"/>
-</signal>
 <signal name="N$19">
 <contactref element="U10" pad="2"/>
@@
 <contactref element="U10" pad="7"/>
 <contactref element="R48" pad="2"/>
-<wire x1="1.8" y1="19.8" x2="1.8" y2="18.82426875" width="0.2032" layer="1"/>
-<wire x1="1.8" y1="18.82426875" x2="2.7207125" y2="17.90355625" width="0.2032" layer="1"/>
+<wire x1="1.8" y1="19.8" x2="1.8" y2="19.22426875" width="0.2032" layer="1"/>
+<wire x1="2.7207125" y1="18.30355625" x2="2.7207125" y2="17.90355625" width="0.2032" layer="1"/>
+<wire x1="2.7207125" y1="18.30355625" x2="1.8" y2="19.22426875" width="0.2032" layer="1"/>
 <wire x1="7.397915625" y1="4.290809375" x2="6.86" y2="3.75289375" width="0.2032" layer="1"/>
 <wire x1="6.86" y1="3.539996875" x2="8.04644375" y2="2.353553125" width="0.2032" layer="1"/>
-<via x="1.8" y="18.82426875" extent="1-16" drill="0.2"/>
+<via x="1.8" y="19.22426875" extent="1-16" drill="0.2"/>
 <wire x1="6.86" y1="3.72" x2="6.86" y2="3.539996875" width="0.2032" layer="1"/>
-<wire x1="1.8" y1="18.82426875" x2="1.8" y2="12.4" width="0.2032" layer="16"/>
-<wire x1="1.8" y1="12.4" x2="5.1079" y2="9.0921" width="0.2032" layer="16"/>
+<wire x1="1.8" y1="19.22426875" x2="1.2" y2="18.62426875" width="0.2032" layer="16"/>
+<wire x1="1.2" y1="14.8" x2="1.2" y2="18.62426875" width="0.2032" layer="16"/>
+<wire x1="5.1079" y1="9.0921" x2="1.7" y2="12.5" width="0.2032" layer="16"/>
 <wire x1="6.86" y1="3.75289375" x2="6.86" y2="3.72" width="0.2032" layer="1"/>
 <via x="6.86" y="3.72" extent="1-16" drill="0.2"/>
@@
 <wire x1="5.78" y1="3.72" x2="6.86" y2="3.72" width="0.2032" layer="16"/>
 <wire x1="5.78" y1="3.72" x2="5.1079" y2="4.3921" width="0.2032" layer="16"/>
+<wire x1="1.7" y1="12.5" x2="1.7" y2="14.3" width="0.2032" layer="16"/>
+<wire x1="1.7" y1="14.3" x2="1.2" y2="14.8" width="0.2032" layer="16"/>
 </signal>
 <signal name="VBAT_REF">
