File: tps65987d/Type-C Test Fixture (TPS65987D)_v3.sch (EAGLE design)
At the start: 195 parts, among them J1 105450-0101, J2 105450-0101, J3 105450-0101, J4 640456-4, J5 5040500491, Q1 AO3400A, Q10 AO3400A, Q11 AO3400A, Q12 AO3400A, Q13 AO3400A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

Commit message: Fix 5V FB resistors
Parts:
- removed R43: 332k, rcl:R-EU_R0402
- removed R44: 1M, rcl:R-EU_R0402
Connections:
- removed net FB: R43.1, R44.1, U10.FB
- net +5V: now also U10.FB; no longer R44.2
- net GND: no longer R43.2
Changed lines of the file:
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@@
 <part name="C68" library="SparkFun-Capacitors" deviceset="1.0UF" device="-0603-16V-10%" value="10uF"/>
 <part name="U$12" library="LCD Driver" deviceset="VSYS" device=""/>
-<part name="R43" library="rcl" deviceset="R-EU_" device="R0402" package3d_urn="urn:adsk.eagle:package:23547/3" value="332k"/>
-<part name="R44" library="rcl" deviceset="R-EU_" device="R0402" package3d_urn="urn:adsk.eagle:package:23547/3" value="1M"/>
 <part name="GND45" library="supply1" deviceset="GND" device=""/>
 <part name="GND46" library="supply1" deviceset="GND" device=""/>
 <part name="GND47" library="supply1" deviceset="GND" device=""/>
 <part name="GND48" library="supply1" deviceset="GND" device=""/>
-<part name="GND49" library="supply1" deviceset="GND" device=""/>
 <part name="GND50" library="supply1" deviceset="GND" device=""/>
 <part name="R48" library="rcl" deviceset="R-EU_" device="R0402" package3d_urn="urn:adsk.eagle:package:23547/3" value="1M"/>
@@
 </instance>
 <instance part="U$12" gate="G$1" x="650.24" y="419.1" smashed="yes"/>
-<instance part="R43" gate="G$1" x="619.76" y="381" smashed="yes" rot="R270">
-<attribute name="NAME" x="615.7214" y="379.73" size="1.778" layer="95" font="vector" rot="R90"/>
-<attribute name="VALUE" x="617.982" y="379.73" size="1.778" layer="96" font="vector" rot="R90"/>
-</instance>
-<instance part="R44" gate="G$1" x="619.76" y="398.78" smashed="yes" rot="R90">
-<attribute name="NAME" x="616.1786" y="400.05" size="1.778" layer="95" font="vector" rot="R270"/>
-<attribute name="VALUE" x="613.918" y="400.05" size="1.778" layer="96" font="vector" rot="R270"/>
-</instance>
 <instance part="GND45" gate="1" x="650.24" y="393.7" smashed="yes">
 <attribute name="VALUE" x="647.7" y="391.16" size="1.778" layer="96" font="vector"/>
@@
 <attribute name="VALUE" x="541.02" y="383.54" size="1.778" layer="96" font="vector"/>
 </instance>
-<instance part="GND49" gate="1" x="619.76" y="370.84" smashed="yes">
-<attribute name="VALUE" x="617.22" y="368.3" size="1.778" layer="96" font="vector"/>
-</instance>
 <instance part="GND50" gate="1" x="568.96" y="388.62" smashed="yes">
 <attribute name="VALUE" x="566.42" y="386.08" size="1.778" layer="96" font="vector"/>
@@
 </segment>
 <segment>
-<pinref part="R43" gate="G$1" pin="2"/>
-<wire x1="619.76" y1="375.92" x2="619.76" y2="373.38" width="0.1524" layer="91"/>
-<pinref part="GND49" gate="1" pin="GND"/>
-</segment>
-<segment>
 <pinref part="U10" gate="G$1" pin="CC"/>
 <wire x1="574.04" y1="396.24" x2="568.96" y2="396.24" width="0.1524" layer="91"/>
@@
 <segment>
 <pinref part="U10" gate="G$1" pin="VOUT"/>
-<wire x1="604.52" y1="406.4" x2="619.76" y2="406.4" width="0.1524" layer="91"/>
+<wire x1="604.52" y1="406.4" x2="629.92" y2="406.4" width="0.1524" layer="91"/>
 <pinref part="C60" gate="G$1" pin="1"/>
-<wire x1="619.76" y1="406.4" x2="629.92" y2="406.4" width="0.1524" layer="91"/>
 <wire x1="629.92" y1="406.4" x2="640.08" y2="406.4" width="0.1524" layer="91"/>
 <junction x="629.92" y="406.4"/>
@@
 <pinref part="U$12" gate="G$1" pin="VSYS"/>
 <wire x1="650.24" y1="406.4" x2="650.24" y2="416.56" width="0.1524" layer="91"/>
-<pinref part="R44" gate="G$1" pin="2"/>
-<wire x1="619.76" y1="403.86" x2="619.76" y2="406.4" width="0.1524" layer="91"/>
-<junction x="619.76" y="406.4"/>
 </segment>
 <segment>
@@
 <label x="576.58" y="434.34" size="1.778" layer="95" font="vector"/>
 </segment>
+<segment>
+<pinref part="U10" gate="G$1" pin="FB"/>
+<wire x1="574.04" y1="406.4" x2="558.8" y2="406.4" width="0.1524" layer="91"/>
+<label x="558.8" y="406.4" size="1.778" layer="95" font="vector"/>
+</segment>
 </net>
 <net name="N$10" class="0">
@@
 </segment>
 </net>
-<net name="FB" class="0">
-<segment>
-<pinref part="U10" gate="G$1" pin="FB"/>
-<wire x1="574.04" y1="406.4" x2="558.8" y2="406.4" width="0.1524" layer="91"/>
-<label x="558.8" y="406.4" size="1.778" layer="95" font="vector"/>
-</segment>
-<segment>
-<pinref part="R44" gate="G$1" pin="1"/>
-<pinref part="R43" gate="G$1" pin="1"/>
-<wire x1="619.76" y1="393.7" x2="619.76" y2="388.62" width="0.1524" layer="91"/>
-<wire x1="619.76" y1="388.62" x2="619.76" y2="386.08" width="0.1524" layer="91"/>
-<wire x1="619.76" y1="388.62" x2="627.38" y2="388.62" width="0.1524" layer="91"/>
-<junction x="619.76" y="388.62"/>
-<label x="624.84" y="388.62" size="1.778" layer="95" font="vector"/>
-</segment>
-</net>
