File: cm5_carrier_pcb/Retro_Lite_CM5_IO_X2.2.sch (EAGLE design)
At the start: 317 parts, among them J1 5025700893, J10 5051100892, J11 1072TR, J12 5034802000, J13 5040500491, J14 5051100492, J2 SJ-43516-SMT, J4 5051100492, J5 685119136923, J6 5034802000, J7 105450-0101, J8 MDT320E01001, J9 5051103091, Q1 AO3400A, Q2 AO3400A, Q3 AO3400A, Q4 AO3400A, Q5 AO3400A, Q6 AO3400A, Q7 AO3400A, Q8 AO3400A, Q9 AO3400A, U10 UM3204QQFN14_3.5X3.5_UM3204_U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, U11 MAX17055ETB+T, U12 SY8089AAACSY8089AAAC_SGY-L, U13 UM3204QQFN14_3.5X3.5_UM3204_U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, U14 MCU-ATTINY84A-MU(QFN20), U16 TPS61160ADRVT, U18 TSIC_306_SOP-8, U19 SN74LVC1G17DCKR, U2 TPD4E05U06DQAR, U20 SN74LVC1G17DCKR, U21 TPS65987DDHRSHR, U22 TPD4E05U06DQAR, U23 TUSB546-DCIRNQT, U24 TPD4E05U06DQAR, U3 TPD4E05U06DQAR, U4 W25X05CLUXIGTR, U5 BQ24292I, U6 WM8960, U7 TPS61235PRWLT, U8 UM3204QQFN14_3.5X3.5_UM3204_U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, U9 UM3204QQFN14_3.5X3.5_UM3204_U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, Y1 ECS-3225MV-240-BN-TR, Y2 ECS-.327-12.5-12R-TR

Commit message: Fix M.2 standoff hole size for 9774015243R
Parts:
- added H1: M2 x 1.5mm, Eagle_WA-SMSI (rev21a):WA-SMSI_9774XXX243_9774015243R
- renumbered LOW_BAT to VBAT_L
Connections:
- net GND: now also H1.1; no longer U$7.HOLE
Other:
- note added: "Indicates succesfful FET switch, charge status & low VBAT."
- note added: "SD Interface"
- note removed: "Indicates succesfful FET switch and charge status."
- note removed: "SD Card"
Changed lines of the file:
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@@
 <part name="J10" library="5051100892" deviceset="5051100892" device=""/>
 <part name="P+4" library="supply1" deviceset="VCC" device=""/>
-<part name="GND37" library="supply1" library_urn="urn:adsk.eagle:library:371" deviceset="GND" device=""/>
 <part name="GPIO_VREF" library="testpad" deviceset="TP" device="TP07R"/>
 <part name="GND41" library="supply1" library_urn="urn:adsk.eagle:library:371" deviceset="GND" device=""/>
@@
 <part name="R57" library="rcl" deviceset="R-EU_" device="R0402" package3d_urn="urn:adsk.eagle:package:23547/3" value="27.4k"/>
 <part name="GND59" library="supply1" deviceset="GND" device=""/>
-<part name="LOW_BAT" library="led" deviceset="LED" device="SML0603"/>
+<part name="VBAT_L" library="led" deviceset="LED" device="SML0603"/>
 <part name="R58" library="rcl" deviceset="R-EU_" device="R0402" package3d_urn="urn:adsk.eagle:package:23547/3" value="2.2k"/>
 <part name="U$42" library="LCD Driver" deviceset="VSYS" device=""/>
@@
 <part name="P+9" library="supply1" library_urn="urn:adsk.eagle:library:371" deviceset="VCC" device=""/>
 <part name="GND105" library="supply1" library_urn="urn:adsk.eagle:library:371" deviceset="GND" device=""/>
+<part name="H1" library="Eagle_WA-SMSI (rev21a)" deviceset="WA-SMSI_9774XXX243" device="_9774015243R" package3d_urn="urn:adsk.eagle:package:14321879/3" value="M2 x 1.5mm"/>
+<part name="GND110" library="supply1" library_urn="urn:adsk.eagle:library:371" deviceset="GND" device=""/>
 </parts>
 <sheets>
@@
 <wire x1="492.76" y1="58.42" x2="492.76" y2="193.04" width="1.016" layer="114"/>
 <wire x1="347.98" y1="58.42" x2="492.76" y2="58.42" width="1.016" layer="114"/>
-<text x="381" y="167.64" size="12.7" layer="114" font="vector">SD Card</text>
+<text x="360.68" y="167.64" size="12.7" layer="114" font="vector">SD Interface</text>
 <wire x1="502.92" y1="58.42" x2="502.92" y2="193.04" width="1.016" layer="114"/>
 <wire x1="502.92" y1="193.04" x2="647.7" y2="193.04" width="1.016" layer="114"/>
@@
 <text x="748.03" y="497.84" size="2.286" layer="97" font="vector" rot="R180">TACH (PWM15_M1) and PWM pins to
 respective PWM pins. </text>
-<text x="853.44" y="497.84" size="1.9304" layer="97" font="vector" rot="R180">Indicates succesfful FET switch
-and charge status. </text>
+<text x="858.52" y="497.84" size="1.9304" layer="97" font="vector" rot="R180">Indicates succesfful FET switch,
+charge status &amp; low VBAT. </text>
 <wire x1="347.98" y1="342.9" x2="347.98" y2="200.66" width="1.016" layer="114"/>
 <wire x1="551.18" y1="342.9" x2="551.18" y2="200.66" width="1.016" layer="114"/>
@@
 <attribute name="VALUE" x="518.16" y="144.78" size="1.778" layer="96" font="vector"/>
 </instance>
-<instance part="LOW_BAT" gate="G$1" x="822.96" y="548.64" smashed="yes">
+<instance part="VBAT_L" gate="G$1" x="822.96" y="548.64" smashed="yes">
 <attribute name="NAME" x="829.056" y="538.988" size="1.778" layer="95" font="vector" rot="R90"/>
 <attribute name="VALUE" x="828.675" y="544.068" size="1.778" layer="96" rot="R90"/>
@@
 </segment>
 <segment>
-<pinref part="LOW_BAT" gate="G$1" pin="A"/>
+<pinref part="VBAT_L" gate="G$1" pin="A"/>
 <wire x1="822.96" y1="551.18" x2="822.96" y2="553.72" width="0.1524" layer="91"/>
 <label x="825.5" y="558.8" size="1.778" layer="95" font="vector" rot="R180"/>
@@
 <net name="N$54" class="0">
 <segment>
-<pinref part="LOW_BAT" gate="G$1" pin="C"/>
+<pinref part="VBAT_L" gate="G$1" pin="C"/>
 <pinref part="R58" gate="G$1" pin="2"/>
 <wire x1="822.96" y1="543.56" x2="822.96" y2="541.02" width="0.1524" layer="91"/>
@@
 </instance>
 <instance part="P+4" gate="VCC" x="180.34" y="185.42" smashed="yes"/>
-<instance part="GND37" gate="1" x="142.24" y="58.42" smashed="yes">
-<attribute name="VALUE" x="139.7" y="53.34" size="1.778" layer="96" font="vector"/>
-</instance>
 <instance part="C43" gate="G$1" x="266.7" y="579.12" smashed="yes" rot="R180">
 <attribute name="NAME" x="265.176" y="578.739" size="1.778" layer="95" font="vector" rot="R180"/>
@@
 </instance>
 <instance part="U$24" gate="G$1" x="772.16" y="543.56" smashed="yes"/>
+<instance part="H1" gate="G$1" x="281.94" y="180.34" smashed="yes" rot="R90">
+<attribute name="NAME" x="278.384" y="180.34" size="1.27" layer="95" rot="R90" align="bottom-center"/>
+<attribute name="VALUE" x="286.512" y="177.292" size="1.27" layer="95" rot="R90"/>
+</instance>
+<instance part="GND110" gate="1" x="281.94" y="167.64" smashed="yes">
+<attribute name="VALUE" x="279.4" y="162.56" size="1.778" layer="96" font="vector"/>
+</instance>
 </instances>
 <busses>
@@
 </segment>
 <segment>
-<pinref part="U$7" gate="G$1" pin="HOLE"/>
-<wire x1="142.24" y1="76.2" x2="142.24" y2="60.96" width="0.1524" layer="91"/>
-<pinref part="GND37" gate="1" pin="GND"/>
-</segment>
-<segment>
 <pinref part="C48" gate="G$1" pin="1"/>
 <pinref part="C45" gate="G$1" pin="1"/>
@@
 <pinref part="GND31" gate="1" pin="GND"/>
 </segment>
+<segment>
+<pinref part="H1" gate="G$1" pin="1"/>
+<wire x1="281.94" y1="175.26" x2="281.94" y2="170.18" width="0.1524" layer="91"/>
+<pinref part="GND110" gate="1" pin="GND"/>
+</segment>
 </net>

Commit message: Add BG_STAT, PG_GOOD pins to CM5 GPIOs
Parts:
- removed PCIE_USB_N, PCIE_USB_P, USB20_HOST1_N, USB20_HOST1_P: TPTP07R, testpad:TPTP07R
- added BMS_INT: TPTP07R, testpad:TPTP07R
- added PG: (no value), led:LEDSML0603
- added R59: 4.7k, rcl:R-EU_R0402
- added R69: 2.2k, rcl:R-EU_R0402
Connections:
- removed net GPIO17_INT: R53.2, U11.ALRT
- removed net GPIO1_A6_CAM1_E: U9.B3
- removed net WIFI_USB_N: J8.5, PCIE_USB_N.TP
- removed net WIFI_USB_P: J8.3, PCIE_USB_P.TP
- new net BMS_INT: BMS_INT.TP, R59.2, U5.INT
- new net BMS_PG: R69.1
- new net N$66: PG.C, R69.2
- net BMS_STAT: now also U9.B3
- net GPIO0_C7: now also U5.PG
- net GPIO1_C4: now also R53.2, U11.ALRT
- net I2C8_SCL_M2: no longer R48.1
- net I2C8_SCL_M2_CAM: now also R48.1
- net I2C8_SDA_M2: no longer R52.1
- net I2C8_SDA_M2_CAM: now also R52.1
- net USB20_HOST1_D_N: now also J8.5; no longer USB20_HOST1_N.TP
- net USB20_HOST1_D_P: now also J8.3; no longer USB20_HOST1_P.TP
- net VSYS: now also PG.A, R59.1
Other:
- note added: "Checked battery polartiy. OK! I2C pins already have pull-ups on CM5 board."
- note added: "For sleep mode/shutdown & low voltage notification."
- note removed: "Checked battery polartiy. OK! I2C pins already have pull-ups."
- moved on the sheet: R48, R52
