File: cm5_carrier_pcb/RetroLiteCM5IOFinal_v2.sch (EAGLE design)
At the start: 327 parts, among them J1 5025700893, J10 5051100892, J11 1072TR, J12 5034802000, J13 5040500491, J14 5051100492, J2 SJ-43516-SMT, J4 5051100492, J5 685119136923, J6 5034802000, J7 105450-0101, J8 MDT320E01001, J9 5051103091, Q1 AO3400A, Q2 AO3400A, Q3 AO3400A, Q4 AO3400A, Q5 AO3400A, Q6 AO3400A, Q7 AO3400A, Q8 AO3400A, Q9 AO3400A, U10 UM3204QQFN14_3.5X3.5_UM3204_U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, U11 MAX17055ETB+T, U12 SY8089AAACSY8089AAAC_SGY-L, U13 UM3204QQFN14_3.5X3.5_UM3204_U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, U14 MCU-ATTINY84A-MU(QFN20), U16 TPS61160ADRVT, U18 TSIC_306_SOP-8, U2 TPD4E05U06DQAR, U21 TPS65987DDHRSHR, U22 TPD4E05U06DQAR, U23 TUSB546-DCIRNQT, U24 TPD4E05U06DQAR, U3 TPD4E05U06DQAR, U4 W25X05CLUXIGTR, U5 BQ24292I, U6 WM8960, U7 TPS61235PRWLT, U8 UM3204QQFN14_3.5X3.5_UM3204_U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, U9 UM3204QQFN14_3.5X3.5_UM3204_U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, Y1 ECS-3225MV-240-BN-TR, Y2 ECS-.327-12.5-12R-TR

Commit message: Flip TPS65987D jumper clock/data (I2C)
Connections:
- new net I2C2_IRQ: U21.!I2C2_IRQ
- new net I2C3_IRQ: U21.!I2C3_IRQ!(GPIO7)
- new net N$69: U21.I2C2_SCL
- new net N$70: U21.I2C2_SDA
- net I2C1_SCL: now also R73.2; no longer R70.2
- net I2C1_SDA: now also R70.2; no longer R73.2
Changed lines of the file:
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@@
+</segment>
+<segment>
+<pinref part="R73" gate="G$1" pin="2"/>
+<wire x1="274.32" y1="358.14" x2="274.32" y2="365.76" width="0.1524" layer="91"/>
+<label x="274.32" y="358.14" size="1.778" layer="95" font="vector" rot="R90"/>
+</segment>
+</net>
+<net name="I2C1_SDA" class="0">
+<segment>
+<pinref part="U21" gate="G$1" pin="I2C1_SDA"/>
+<wire x1="167.64" y1="368.3" x2="187.96" y2="368.3" width="0.1524" layer="91"/>
+<label x="182.88" y="368.3" size="1.778" layer="95" font="vector"/>
+</segment>
+<segment>
+<pinref part="R72" gate="G$1" pin="1"/>
+<wire x1="256.54" y1="347.98" x2="256.54" y2="340.36" width="0.1524" layer="91"/>
+<label x="256.54" y="335.28" size="1.778" layer="95" font="vector" rot="R90"/>
 </segment>
 <segment>
@@
 <wire x1="266.7" y1="358.14" x2="266.7" y2="365.76" width="0.1524" layer="91"/>
 <label x="266.7" y="358.14" size="1.778" layer="95" font="vector" rot="R90"/>
-</segment>
-</net>
-<net name="I2C1_SDA" class="0">
-<segment>
-<pinref part="U21" gate="G$1" pin="I2C1_SDA"/>
-<wire x1="167.64" y1="368.3" x2="187.96" y2="368.3" width="0.1524" layer="91"/>
-<label x="182.88" y="368.3" size="1.778" layer="95" font="vector"/>
-</segment>
-<segment>
-<pinref part="R72" gate="G$1" pin="1"/>
-<wire x1="256.54" y1="347.98" x2="256.54" y2="340.36" width="0.1524" layer="91"/>
-<label x="256.54" y="335.28" size="1.778" layer="95" font="vector" rot="R90"/>
-</segment>
-<segment>
-<pinref part="R73" gate="G$1" pin="2"/>
-<wire x1="274.32" y1="358.14" x2="274.32" y2="365.76" width="0.1524" layer="91"/>
-<label x="274.32" y="358.14" size="1.778" layer="95" font="vector" rot="R90"/>
 </segment>
 </net>
@@
 </segment>
 </net>
+<net name="I2C2_IRQ" class="0">
+<segment>
+<pinref part="U21" gate="G$1" pin="!I2C2_IRQ"/>
+<wire x1="167.64" y1="363.22" x2="187.96" y2="363.22" width="0.1524" layer="91"/>
+<label x="182.88" y="363.22" size="1.778" layer="95"/>
+</segment>
+</net>
+<net name="N$69" class="0">
+<segment>
+<pinref part="U21" gate="G$1" pin="I2C2_SCL"/>
+<wire x1="167.64" y1="360.68" x2="187.96" y2="360.68" width="0.1524" layer="91"/>
+</segment>
+</net>
+<net name="N$70" class="0">
+<segment>
+<pinref part="U21" gate="G$1" pin="I2C2_SDA"/>
+<wire x1="167.64" y1="358.14" x2="187.96" y2="358.14" width="0.1524" layer="91"/>
+</segment>
+</net>
+<net name="I2C3_IRQ" class="0">
+<segment>
+<pinref part="U21" gate="G$1" pin="!I2C3_IRQ!(GPIO7)"/>
+<wire x1="167.64" y1="350.52" x2="187.96" y2="350.52" width="0.1524" layer="91"/>
+<label x="182.88" y="350.52" size="1.778" layer="95" font="vector"/>
+</segment>
+</net>
